File: hardware/design/BLDC_4.5/hall_filters.sch (KiCad schematic (older format))
At the start: 11 parts

Commit message: Layout updated. Added inner power planes, changed USB connector, added CAN transceiver and connector, added 3D models copper pour under the mosfets and references moved to visible places
Signed-off-by: Marcos Chaparro <marcos@mrkindustries.com.ar>
Parts:
- C4, C5, C6, C7: footprint (none) -> SMD_Packages:SMD-0603_c
- R10, R11, R12, R13, R7, R8, R9: footprint (none) -> SMD_Packages:SMD-0603_r
Changed lines of the file:
@@
 F 0 "R7" V 4850 3400 50  0000 C CNN
 F 1 "10k" V 4900 3200 50  0000 C CNN
-F 2 "" H 4900 3200 60  0001 C CNN
+F 2 "SMD_Packages:SMD-0603_r" H 4900 3200 60  0001 C CNN
 F 3 "" H 4900 3200 60  0001 C CNN
 	1    4900 3200
@@
 F 0 "R8" V 5500 3950 50  0000 C CNN
 F 1 "10k" V 5550 3750 50  0000 C CNN
-F 2 "" H 5550 3750 60  0001 C CNN
+F 2 "SMD_Packages:SMD-0603_r" H 5550 3750 60  0001 C CNN
 F 3 "" H 5550 3750 60  0001 C CNN
 	1    5550 3750
@@
 F 0 "R9" V 5500 3850 50  0000 C CNN
 F 1 "10k" V 5550 3650 50  0000 C CNN
-F 2 "" H 5550 3650 60  0001 C CNN
+F 2 "SMD_Packages:SMD-0603_r" H 5550 3650 60  0001 C CNN
 F 3 "" H 5550 3650 60  0001 C CNN
 	1    5550 3650
@@
 F 0 "R10" V 5500 3750 50  0000 C CNN
 F 1 "10k" V 5550 3550 50  0000 C CNN
-F 2 "" H 5550 3550 60  0001 C CNN
+F 2 "SMD_Packages:SMD-0603_r" H 5550 3550 60  0001 C CNN
 F 3 "" H 5550 3550 60  0001 C CNN
 	1    5550 3550
@@
 F 0 "C5" H 6000 4350 50  0000 L CNN
 F 1 "4n7" H 6000 4150 50  0000 L CNN
-F 2 "" H 5950 4250 60  0001 C CNN
+F 2 "SMD_Packages:SMD-0603_c" H 5950 4250 60  0001 C CNN
 F 3 "" H 5950 4250 60  0001 C CNN
 	1    5950 4250
@@
 F 0 "C6" H 6250 4350 50  0000 L CNN
 F 1 "4n7" H 6250 4150 50  0000 L CNN
-F 2 "" H 6200 4250 60  0001 C CNN
+F 2 "SMD_Packages:SMD-0603_c" H 6200 4250 60  0001 C CNN
 F 3 "" H 6200 4250 60  0001 C CNN
 	1    6200 4250
@@
 F 0 "C7" H 6500 4350 50  0000 L CNN
 F 1 "4n7" H 6500 4150 50  0000 L CNN
-F 2 "" H 6450 4250 60  0001 C CNN
+F 2 "SMD_Packages:SMD-0603_c" H 6450 4250 60  0001 C CNN
 F 3 "" H 6450 4250 60  0001 C CNN
 	1    6450 4250
@@
 $EndComp
 $Comp
-L GND #PWR503
+L GND #PWR033
 U 1 1 53FBB5B2
 P 5950 4450
-F 0 "#PWR503" H 5950 4450 30  0001 C CNN
+F 0 "#PWR033" H 5950 4450 30  0001 C CNN
 F 1 "GND" H 5950 4380 30  0001 C CNN
 F 2 "" H 5950 4450 60  0001 C CNN
@@
 F 0 "R11" V 4950 3400 50  0000 C CNN
 F 1 "2k2" V 5000 3200 50  0000 C CNN
-F 2 "" H 5000 3200 60  0001 C CNN
+F 2 "SMD_Packages:SMD-0603_r" H 5000 3200 60  0001 C CNN
 F 3 "" H 5000 3200 60  0001 C CNN
 	1    5000 3200
@@
 F 0 "R12" V 5050 3400 50  0000 C CNN
 F 1 "2k2" V 5100 3200 50  0000 C CNN
-F 2 "" H 5100 3200 60  0001 C CNN
+F 2 "SMD_Packages:SMD-0603_r" H 5100 3200 60  0001 C CNN
 F 3 "" H 5100 3200 60  0001 C CNN
 	1    5100 3200
@@
 F 0 "R13" V 5150 3400 50  0000 C CNN
 F 1 "2k2" V 5200 3200 50  0000 C CNN
-F 2 "" H 5200 3200 60  0001 C CNN
+F 2 "SMD_Packages:SMD-0603_r" H 5200 3200 60  0001 C CNN
 F 3 "" H 5200 3200 60  0001 C CNN
 	1    5200 3200
@@
 F 0 "C4" H 5150 4350 50  0000 L CNN
 F 1 "4n7" H 5150 4150 50  0000 L CNN
-F 2 "" H 5100 4250 60  0001 C CNN
+F 2 "SMD_Packages:SMD-0603_c" H 5100 4250 60  0001 C CNN
 F 3 "" H 5100 4250 60  0001 C CNN
 	1    5100 4250
@@
 $EndComp
 $Comp
-L GND #PWR502
+L GND #PWR034
 U 1 1 53FBB5D4
 P 5100 4450
-F 0 "#PWR502" H 5100 4450 30  0001 C CNN
+F 0 "#PWR034" H 5100 4450 30  0001 C CNN
 F 1 "GND" H 5100 4380 30  0001 C CNN
 F 2 "" H 5100 4450 60  0001 C CNN
@@
 $EndComp
 $Comp
-L VCC #PWR501
+L VCC #PWR035
 U 1 1 53FBB5DA
 P 4900 2850
-F 0 "#PWR501" H 4900 2950 30  0001 C CNN
+F 0 "#PWR035" H 4900 2950 30  0001 C CNN
 F 1 "VCC" V 4850 2900 30  0000 C CNN
 F 2 "" H 4900 2850 60  0001 C CNN
@@
 	5100 3850 5100 4050
 $Comp
-L GND #PWR504
+L GND #PWR036
 U 1 1 53FBB5F9
 P 6200 4450
-F 0 "#PWR504" H 6200 4450 30  0001 C CNN
+F 0 "#PWR036" H 6200 4450 30  0001 C CNN
 F 1 "GND" H 6200 4380 30  0001 C CNN
 F 2 "" H 6200 4450 60  0001 C CNN
@@
 $EndComp
 $Comp
-L GND #PWR505
+L GND #PWR037
 U 1 1 53FBB5FF
 P 6450 4450
-F 0 "#PWR505" H 6450 4450 30  0001 C CNN
+F 0 "#PWR037" H 6450 4450 30  0001 C CNN
 F 1 "GND" H 6450 4380 30  0001 C CNN
 F 2 "" H 6450 4450 60  0001 C CNN
