File: hardware/design/BLDC_4.5/mosfets.sch (KiCad schematic (older format))
At the start: 15 parts, among them Q1 IRFS3006, Q2 IRFS3006, Q3 IRFS3006, Q4 IRFS3006, Q5 IRFS3006, Q6 IRFS3006

Commit message: Layout updated. Added inner power planes, changed USB connector, added CAN transceiver and connector, added 3D models copper pour under the mosfets and references moved to visible places
Signed-off-by: Marcos Chaparro <marcos@mrkindustries.com.ar>
Parts:
- Q1, Q2, Q3, Q4, Q5, Q6: footprint (none) -> CRF1:D2PAK-7-GDS
- R28, R29, R30, R34, R35, R36, R42, R43, R46: footprint (none) -> SMD_Packages:SMD-0603_r
Changed lines of the file:
@@
 $Descr A4 11693 8268
 encoding utf-8
-Sheet 3 7
+Sheet 2 7
 Title "BLDC Driver 4.5"
 Date "25 Aug 2014"
@@
 F 0 "R46" V 7950 4050 50  0000 C CNN
 F 1 "33k" V 7850 4050 50  0000 C CNN
-F 2 "" H 7850 4050 60  0001 C CNN
+F 2 "SMD_Packages:SMD-0603_r" H 7850 4050 60  0001 C CNN
 F 3 "" H 7850 4050 60  0001 C CNN
 	1    7850 4050
@@
 F 0 "R30" V 4500 4050 50  0000 C CNN
 F 1 "33k" V 4400 4050 50  0000 C CNN
-F 2 "" H 4400 4050 60  0001 C CNN
+F 2 "SMD_Packages:SMD-0603_r" H 4400 4050 60  0001 C CNN
 F 3 "" H 4400 4050 60  0001 C CNN
 	1    4400 4050
@@
 F 0 "Q1" H 4960 2970 60  0000 R CNN
 F 1 "IRFS3006" V 5150 2950 60  0000 R CNN
-F 2 "" H 4950 2800 60  0001 C CNN
+F 2 "CRF1:D2PAK-7-GDS" H 4950 2800 60  0001 C CNN
 F 3 "" H 4950 2800 60  0001 C CNN
 	1    4950 2800
@@
 F 0 "Q2" H 4960 3920 60  0000 R CNN
 F 1 "IRFS3006" V 5150 4050 60  0000 R CNN
-F 2 "" H 4950 3750 60  0001 C CNN
+F 2 "CRF1:D2PAK-7-GDS" H 4950 3750 60  0001 C CNN
 F 3 "" H 4950 3750 60  0001 C CNN
 	1    4950 3750
@@
 F 0 "R29" V 4500 3750 50  0000 C CNN
 F 1 "4R7" V 4400 3750 50  0000 C CNN
-F 2 "" H 4400 3750 60  0001 C CNN
+F 2 "SMD_Packages:SMD-0603_r" H 4400 3750 60  0001 C CNN
 F 3 "" H 4400 3750 60  0001 C CNN
 	1    4400 3750
@@
 F 0 "R28" V 4500 2800 50  0000 C CNN
 F 1 "4R7" V 4400 2800 50  0000 C CNN
-F 2 "" H 4400 2800 60  0001 C CNN
+F 2 "SMD_Packages:SMD-0603_r" H 4400 2800 60  0001 C CNN
 F 3 "" H 4400 2800 60  0001 C CNN
 	1    4400 2800
@@
 F 0 "R34" V 6050 2800 50  0000 C CNN
 F 1 "4R7" V 5950 2800 50  0000 C CNN
-F 2 "" H 5950 2800 60  0001 C CNN
+F 2 "SMD_Packages:SMD-0603_r" H 5950 2800 60  0001 C CNN
 F 3 "" H 5950 2800 60  0001 C CNN
 	1    5950 2800
@@
 F 0 "R35" V 6050 3750 50  0000 C CNN
 F 1 "4R7" V 5950 3750 50  0000 C CNN
-F 2 "" H 5950 3750 60  0001 C CNN
+F 2 "SMD_Packages:SMD-0603_r" H 5950 3750 60  0001 C CNN
 F 3 "" H 5950 3750 60  0001 C CNN
 	1    5950 3750
@@
 F 0 "Q4" H 6510 3920 60  0000 R CNN
 F 1 "IRFS3006" V 6700 4050 60  0000 R CNN
-F 2 "" H 6500 3750 60  0001 C CNN
+F 2 "CRF1:D2PAK-7-GDS" H 6500 3750 60  0001 C CNN
 F 3 "" H 6500 3750 60  0001 C CNN
 	1    6500 3750
@@
 F 0 "Q3" H 6510 2970 60  0000 R CNN
 F 1 "IRFS3006" V 6700 2850 60  0000 R CNN
-F 2 "" H 6500 2800 60  0001 C CNN
+F 2 "CRF1:D2PAK-7-GDS" H 6500 2800 60  0001 C CNN
 F 3 "" H 6500 2800 60  0001 C CNN
 	1    6500 2800
@@
 F 0 "Q5" H 8110 2970 60  0000 R CNN
 F 1 "IRFS3006" V 8300 2900 60  0000 R CNN
-F 2 "" H 8100 2800 60  0001 C CNN
+F 2 "CRF1:D2PAK-7-GDS" H 8100 2800 60  0001 C CNN
 F 3 "" H 8100 2800 60  0001 C CNN
 	1    8100 2800
@@
 F 0 "Q6" H 8110 3920 60  0000 R CNN
 F 1 "IRFS3006" V 8300 4000 60  0000 R CNN
-F 2 "" H 8100 3750 60  0001 C CNN
+F 2 "CRF1:D2PAK-7-GDS" H 8100 3750 60  0001 C CNN
 F 3 "" H 8100 3750 60  0001 C CNN
 	1    8100 3750
@@
 F 0 "R43" V 7650 3750 50  0000 C CNN
 F 1 "4R7" V 7550 3750 50  0000 C CNN
-F 2 "" H 7550 3750 60  0001 C CNN
+F 2 "SMD_Packages:SMD-0603_r" H 7550 3750 60  0001 C CNN
 F 3 "" H 7550 3750 60  0001 C CNN
 	1    7550 3750
@@
 F 0 "R42" V 7650 2800 50  0000 C CNN
 F 1 "4R7" V 7550 2800 50  0000 C CNN
-F 2 "" H 7550 2800 60  0001 C CNN
+F 2 "SMD_Packages:SMD-0603_r" H 7550 2800 60  0001 C CNN
 F 3 "" H 7550 2800 60  0001 C CNN
 	1    7550 2800
@@
 F 0 "R36" V 5850 4050 50  0000 C CNN
 F 1 "33k" V 5950 4050 50  0000 C CNN
-F 2 "" H 5950 4050 60  0001 C CNN
+F 2 "SMD_Packages:SMD-0603_r" H 5950 4050 60  0001 C CNN
 F 3 "" H 5950 4050 60  0001 C CNN
 	1    5950 4050
@@
 $EndComp
 $Comp
-L PWR_FLAG #FLG201
+L PWR_FLAG #FLG023
 U 1 1 53F8E6AD
 P 4800 2350
-F 0 "#FLG201" H 4800 2445 30  0001 C CNN
+F 0 "#FLG023" H 4800 2445 30  0001 C CNN
 F 1 "PWR_FLAG" H 4800 2530 30  0000 C CNN
 F 2 "" H 4800 2350 60  0001 C CNN
@@
 $Bitmap
 Pos 2050 6450
-Scale 1.000000
+Scale 1,000000
 Data
 89 50 4E 47 0D 0A 1A 0A 00 00 00 0D 49 48 44 52 00 00 03 8B 00 00 01 56 08 02 00 00 00 4F 4E 9F
@@
 F8 14 F0 0B 42 92 4F 42 07 35 54 00 00 00 00 00 00 7A 11 BC 6D 0C 00 00 00 00 00 F4 2D 50 43 05
 00 00 00 00 00 7D 0B D4 50 01 00 00 00 00 40 DF 02 35 54 00 00 00 00 00 D0 B7 FC 1F 55 28 1C 02
-4B 67 87 83 00 00 00 00 49 45 4E 44 AE 42 60 82 F0
+4B 67 87 83 00 00 00 00 49 45 4E 44 AE 42 60 82 00
 EndData
 $EndBitmap
 $Bitmap
 Pos 10150 5600
-Scale 1.000000
+Scale 1,000000
 Data
 89 50 4E 47 0D 0A 1A 0A 00 00 00 0D 49 48 44 52 00 00 02 72 00 00 02 1A 08 02 00 00 00 2B EB 37
@@
 00 00 00 41 83 58 05 00 00 08 1A C4 2A 00 00 40 D0 20 56 01 00 00 82 06 B1 0A 00 00 10 34 88 55
 00 00 80 A0 41 AC 02 00 00 04 CD FF 03 15 B2 0E 9E 1D 9F E2 F2 00 00 00 00 49 45 4E 44 AE 42 60
-82 46
+82 00
 EndData
 $EndBitmap
 $Bitmap
 Pos 6000 6850
-Scale 1.000000
+Scale 1,000000
 Data
 89 50 4E 47 0D 0A 1A 0A 00 00 00 0D 49 48 44 52 00 00 02 31 00 00 02 30 08 02 00 00 00 F8 51 AD
@@
 6D 12 06 83 C1 60 DA 0B D8 26 61 30 18 0C A6 BD 80 6D 12 06 83 C1 60 DA 0B D8 26 61 30 18 0C A6
 BD 80 6D 12 06 83 C1 60 DA 0B FF 03 68 C2 AC 3A A9 DC 0C E9 00 00 00 00 49 45 4E 44 AE 42 60 82
-78
+00
 EndData
 $EndBitmap
 $Bitmap
 Pos 4350 6700
-Scale 1.000000
+Scale 1,000000
 Data
 89 50 4E 47 0D 0A 1A 0A 00 00 00 0D 49 48 44 52 00 00 01 C1 00 00 01 D6 08 02 00 00 00 80 0A A5
@@
 50 A9 E8 5E 5D 3A 9D 4E 20 10 38 47 FD BC E9 C5 23 08 52 5C 54 54 5F 5F 3F 46 5C 9C 4C 26 63 A3
 F8 9F 0A E6 43 31 30 BE 81 FA D0 5F 5D 10 8C 7F 13 D8 9A 12 06 06 06 06 EF 60 3E 14 03 03 03 83
-77 FE 07 75 CC 31 C3 52 8F 7C 35 00 00 00 00 49 45 4E 44 AE 42 60 82 00
+77 FE 07 75 CC 31 C3 52 8F 7C 35 00 00 00 00 49 45 4E 44 AE 42 60 82 55
 EndData
 $EndBitmap
 $Bitmap
 Pos 2100 2150
-Scale 2.000000
+Scale 2,000000
 Data
 89 50 4E 47 0D 0A 1A 0A 00 00 00 0D 49 48 44 52 00 00 01 C2 00 00 01 99 08 02 00 00 00 95 33 A6
@@
 40 20 9C 12 44 46 09 04 02 E1 94 20 EE F7 67 02 30 C1 25 10 08 E7 25 24 1A 25 10 08 84 53 82 2C
 11 21 10 08 84 53 82 44 A3 04 02 81 70 4A 10 19 25 10 08 84 53 82 C8 28 81 40 20 9C 12 FF 1F 3E
-01 30 64 8D 18 65 07 00 00 00 00 49 45 4E 44 AE 42 60 82 07
+01 30 64 8D 18 65 07 00 00 00 00 49 45 4E 44 AE 42 60 82 FD
 EndData
 $EndBitmap
