File: hardware/design/BLDC/BLDC_4.kicad_pcb (KiCad board)
At the start: 4 copper layers, 38.5 x 59 mm, 128 parts, among them K1 SERVO, P1 HALL/Encoder, P101 CANBUS, P2 SWD, P3 PWR_COMM, P4 IN+, P5 IN-, P6 MOTOR1, P7 MOTOR2, P9 MOTOR3, Q1 IRFS3006, Q2 IRFS3006, Q3 IRFS3006, Q4 IRFS3006, Q5 IRFS3006, Q6 IRFS3006, U1 STM32F40X_LQFP64, U2 NCP1117ST33T3G, U3 DRV8302, U301 LM73, U401 SN65HVD232, X1 MINI-USB-SHIELD-32005-201, X2 8MHz 10ppm

Commit message: Generated and added gerber files
Other:
- board text removed: "Changelog: * Pin4 of the regulator is now pin 2 for better heatsinking * Layer stackup changed to have an inner VDD power plane * Changed USB connector * Added CAN transceiver * Added CAN connector * Added 3D models"
