File: design/CAN.sch (KiCad schematic (older format))
At the start: 4 parts, among them U401 SN65HVD232

Commit message: HW4.8: better shunt routing, extra pin on comm connector, footprint fixed, zone fixes, many other improvements
Parts:
- C401: footprint SMD_Packages:SMD-0402 -> CRF1:SMD-0603_c; symbol C -> C-RESCUE-BLDC_4
- R401, R402: footprint SMD_Packages:SMD-0603_r -> CRF1:SMD-0603_r; symbol R -> R-RESCUE-BLDC_4
- U401: footprint SMD_Packages:SOIC-8-W -> CRF1:SOIC-8-W; symbol MCP2551-I/SN -> MCP2551-I/SN-RESCUE-BLDC_4
Changed lines of the file:
@@
 EESchema Schematic File Version 2
+LIBS:BLDC_4-rescue
 LIBS:power
 LIBS:device
@@
 LIBS:crf_1
 LIBS:BLDC_4-cache
-EELAYER 24 0
+EELAYER 25 0
 EELAYER END
 $Descr A4 11693 8268
 encoding utf-8
 Sheet 4 7
-Title "CAN BUS transceiver"
-Date "25 Aug 2014"
-Rev ""
-Comp "Mrk Industries"
+Title "BLDC Driver 4.8"
+Date "21 aug 2015"
+Rev "4.8"
+Comp "Benjamin Vedder"
 Comment1 ""
 Comment2 ""
@@
 $EndDescr
 $Comp
-L MCP2551-I/SN U401
+L MCP2551-I/SN-RESCUE-BLDC_4 U401
 U 1 1 53F59F90
 P 5850 4050
 F 0 "U401" H 5600 4350 40  0000 C CNN
 F 1 "SN65HVD232" H 6100 3750 40  0000 C CNN
-F 2 "SMD_Packages:SOIC-8-W" H 5850 4050 35  0001 C CIN
+F 2 "CRF1:SOIC-8-W" H 5850 4050 35  0001 C CIN
 F 3 "" H 5850 4050 60  0000 C CNN
 	1    5850 4050
@@
 $EndComp
 $Comp
-L GND #PWR025
+L GND-RESCUE-BLDC_4 #PWR025
 U 1 1 53F59F97
 P 5850 4450
@@
 $EndComp
 $Comp
-L C C401
+L C-RESCUE-BLDC_4 C401
 U 1 1 53F59FA3
 P 6150 3400
 F 0 "C401" H 6150 3500 40  0000 L CNN
 F 1 "2.2u" H 6156 3315 40  0000 L CNN
-F 2 "SMD_Packages:SMD-0402" H 6188 3250 30  0001 C CNN
+F 2 "CRF1:SMD-0603_c" H 6188 3250 30  0001 C CNN
 F 3 "" H 6150 3400 60  0000 C CNN
 	1    6150 3400
@@
 $EndComp
 $Comp
-L GND #PWR028
+L GND-RESCUE-BLDC_4 #PWR028
 U 1 1 53F59FB0
 P 6150 3600
@@
 CAN_TX
 $Comp
-L R R401
+L R-RESCUE-BLDC_4 R401
 U 1 1 540030A8
 P 4900 4050
 F 0 "R401" V 4980 4050 40  0000 C CNN
 F 1 "NI" V 4907 4051 40  0000 C CNN
-F 2 "SMD_Packages:SMD-0603_r" V 4830 4050 30  0001 C CNN
+F 2 "CRF1:SMD-0603_r" V 4830 4050 30  0001 C CNN
 F 3 "" H 4900 4050 30  0000 C CNN
 	1    4900 4050
@@
 NoConn ~ 6300 4100
 $Comp
-L R R402
+L R-RESCUE-BLDC_4 R402
 U 1 1 54003136
 P 6400 4600
 F 0 "R402" H 6550 4600 40  0000 C CNN
 F 1 "10k" V 6407 4601 40  0000 C CNN
-F 2 "SMD_Packages:SMD-0603_r" V 6330 4600 30  0001 C CNN
+F 2 "CRF1:SMD-0603_r" V 6330 4600 30  0001 C CNN
 F 3 "" H 6400 4600 30  0000 C CNN
 	1    6400 4600
@@
 	6400 4250 6300 4250
 $Comp
-L GND #PWR029
+L GND-RESCUE-BLDC_4 #PWR029
 U 1 1 5400318B
 P 6400 4850
