File: design/hall_filters.sch (KiCad schematic (older format))
At the start: 11 parts

Commit message: HW4.8: better shunt routing, extra pin on comm connector, footprint fixed, zone fixes, many other improvements
Parts:
- C4, C5, C6, C7: footprint SMD_Packages:SMD-0603_c -> CRF1:SMD-0603_c; symbol C -> C-RESCUE-BLDC_4
- R10, R11, R12, R13, R7, R8, R9: footprint SMD_Packages:SMD-0603_r -> CRF1:SMD-0603_r; symbol R -> R-RESCUE-BLDC_4
Changed lines of the file:
@@
 EESchema Schematic File Version 2
+LIBS:BLDC_4-rescue
 LIBS:power
 LIBS:device
@@
 LIBS:crf_1
 LIBS:BLDC_4-cache
-EELAYER 24 0
+EELAYER 25 0
 EELAYER END
 $Descr A4 11693 8268
 encoding utf-8
 Sheet 5 7
-Title ""
-Date "25 Aug 2014"
-Rev ""
-Comp ""
+Title "BLDC Driver 4.8"
+Date "21 aug 2015"
+Rev "4.8"
+Comp "Benjamin Vedder"
 Comment1 ""
 Comment2 ""
@@
 $EndDescr
 $Comp
-L R R7
+L R-RESCUE-BLDC_4 R7
 U 1 1 53FBB581
 P 4900 3200
 F 0 "R7" V 4850 3400 50  0000 C CNN
 F 1 "10k" V 4900 3200 50  0000 C CNN
-F 2 "SMD_Packages:SMD-0603_r" H 4900 3200 60  0001 C CNN
+F 2 "CRF1:SMD-0603_r" H 4900 3200 60  0001 C CNN
 F 3 "" H 4900 3200 60  0001 C CNN
 	1    4900 3200
@@
 $EndComp
 $Comp
-L R R8
+L R-RESCUE-BLDC_4 R8
 U 1 1 53FBB588
 P 5550 3750
 F 0 "R8" V 5500 3950 50  0000 C CNN
 F 1 "10k" V 5550 3750 50  0000 C CNN
-F 2 "SMD_Packages:SMD-0603_r" H 5550 3750 60  0001 C CNN
+F 2 "CRF1:SMD-0603_r" H 5550 3750 60  0001 C CNN
 F 3 "" H 5550 3750 60  0001 C CNN
 	1    5550 3750
@@
 $EndComp
 $Comp
-L R R9
+L R-RESCUE-BLDC_4 R9
 U 1 1 53FBB58F
 P 5550 3650
 F 0 "R9" V 5500 3850 50  0000 C CNN
 F 1 "10k" V 5550 3650 50  0000 C CNN
-F 2 "SMD_Packages:SMD-0603_r" H 5550 3650 60  0001 C CNN
+F 2 "CRF1:SMD-0603_r" H 5550 3650 60  0001 C CNN
 F 3 "" H 5550 3650 60  0001 C CNN
 	1    5550 3650
@@
 $EndComp
 $Comp
-L R R10
+L R-RESCUE-BLDC_4 R10
 U 1 1 53FBB596
 P 5550 3550
 F 0 "R10" V 5500 3750 50  0000 C CNN
 F 1 "10k" V 5550 3550 50  0000 C CNN
-F 2 "SMD_Packages:SMD-0603_r" H 5550 3550 60  0001 C CNN
+F 2 "CRF1:SMD-0603_r" H 5550 3550 60  0001 C CNN
 F 3 "" H 5550 3550 60  0001 C CNN
 	1    5550 3550
@@
 $EndComp
 $Comp
-L C C5
+L C-RESCUE-BLDC_4 C5
 U 1 1 53FBB59D
 P 5950 4250
 F 0 "C5" H 6000 4350 50  0000 L CNN
 F 1 "4n7" H 6000 4150 50  0000 L CNN
-F 2 "SMD_Packages:SMD-0603_c" H 5950 4250 60  0001 C CNN
+F 2 "CRF1:SMD-0603_c" H 5950 4250 60  0001 C CNN
 F 3 "" H 5950 4250 60  0001 C CNN
 	1    5950 4250
@@
 $EndComp
 $Comp
-L C C6
+L C-RESCUE-BLDC_4 C6
 U 1 1 53FBB5A4
 P 6200 4250
 F 0 "C6" H 6250 4350 50  0000 L CNN
 F 1 "4n7" H 6250 4150 50  0000 L CNN
-F 2 "SMD_Packages:SMD-0603_c" H 6200 4250 60  0001 C CNN
+F 2 "CRF1:SMD-0603_c" H 6200 4250 60  0001 C CNN
 F 3 "" H 6200 4250 60  0001 C CNN
 	1    6200 4250
@@
 $EndComp
 $Comp
-L C C7
+L C-RESCUE-BLDC_4 C7
 U 1 1 53FBB5AB
 P 6450 4250
 F 0 "C7" H 6500 4350 50  0000 L CNN
 F 1 "4n7" H 6500 4150 50  0000 L CNN
-F 2 "SMD_Packages:SMD-0603_c" H 6450 4250 60  0001 C CNN
+F 2 "CRF1:SMD-0603_c" H 6450 4250 60  0001 C CNN
 F 3 "" H 6450 4250 60  0001 C CNN
 	1    6450 4250
@@
 $EndComp
 $Comp
-L GND #PWR030
+L GND-RESCUE-BLDC_4 #PWR030
 U 1 1 53FBB5B2
 P 5950 4450
@@
 $EndComp
 $Comp
-L R R11
+L R-RESCUE-BLDC_4 R11
 U 1 1 53FBB5B8
 P 5000 3200
 F 0 "R11" V 4950 3400 50  0000 C CNN
 F 1 "2k2" V 5000 3200 50  0000 C CNN
-F 2 "SMD_Packages:SMD-0603_r" H 5000 3200 60  0001 C CNN
+F 2 "CRF1:SMD-0603_r" H 5000 3200 60  0001 C CNN
 F 3 "" H 5000 3200 60  0001 C CNN
 	1    5000 3200
@@
 $EndComp
 $Comp
-L R R12
+L R-RESCUE-BLDC_4 R12
 U 1 1 53FBB5BF
 P 5100 3200
 F 0 "R12" V 5050 3400 50  0000 C CNN
 F 1 "2k2" V 5100 3200 50  0000 C CNN
-F 2 "SMD_Packages:SMD-0603_r" H 5100 3200 60  0001 C CNN
+F 2 "CRF1:SMD-0603_r" H 5100 3200 60  0001 C CNN
 F 3 "" H 5100 3200 60  0001 C CNN
 	1    5100 3200
@@
 $EndComp
 $Comp
-L R R13
+L R-RESCUE-BLDC_4 R13
 U 1 1 53FBB5C6
 P 5200 3200
 F 0 "R13" V 5150 3400 50  0000 C CNN
 F 1 "2k2" V 5200 3200 50  0000 C CNN
-F 2 "SMD_Packages:SMD-0603_r" H 5200 3200 60  0001 C CNN
+F 2 "CRF1:SMD-0603_r" H 5200 3200 60  0001 C CNN
 F 3 "" H 5200 3200 60  0001 C CNN
 	1    5200 3200
@@
 $EndComp
 $Comp
-L C C4
+L C-RESCUE-BLDC_4 C4
 U 1 1 53FBB5CD
 P 5100 4250
 F 0 "C4" H 5150 4350 50  0000 L CNN
 F 1 "4n7" H 5150 4150 50  0000 L CNN
-F 2 "SMD_Packages:SMD-0603_c" H 5100 4250 60  0001 C CNN
+F 2 "CRF1:SMD-0603_c" H 5100 4250 60  0001 C CNN
 F 3 "" H 5100 4250 60  0001 C CNN
 	1    5100 4250
@@
 $EndComp
 $Comp
-L GND #PWR031
+L GND-RESCUE-BLDC_4 #PWR031
 U 1 1 53FBB5D4
 P 5100 4450
@@
 	5100 3850 5100 4050
 $Comp
-L GND #PWR033
+L GND-RESCUE-BLDC_4 #PWR033
 U 1 1 53FBB5F9
 P 6200 4450
@@
 $EndComp
 $Comp
-L GND #PWR034
+L GND-RESCUE-BLDC_4 #PWR034
 U 1 1 53FBB5FF
 P 6450 4450
